File: hard/proj/controller.kicad_pcb (KiCad board)
At the start: 2 copper layers, 44 parts, among them J1 microUSB, J2 EXT1, J3 EXT2, J4 EXT3, J5 EXT4, J6 UART, Q1 BC848B, Q2 BC848B, Q3 BC848B, Q4 BC848B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

Commit message: some PCB
Parts:
- added REF**: MountingHole_3mm_Pad_Via, Mounting_Holes:MountingHole_3mm_Pad_Via, F.Cu at (52.0, 126.0)
- added REF**: MountingHole_3mm_Pad_Via, Mounting_Holes:MountingHole_3mm_Pad_Via, F.Cu at (52.0, 58.0)
- moved R9 164.0 mm to (86.0, 185.0)
- moved J5 162.8 mm to (55.0, 119.0)
- moved R7 160.7 mm to (91.0, 176.0)
- moved R11 158.1 mm to (114.0, 171.0), turned to 180 degrees
- moved D1 157.6 mm to (80.0, 182.0), turned to 180 degrees
- moved Q4 156.3 mm to (122.0, 188.0)
- moved R12 154.3 mm to (114.0, 179.0), turned to 180 degrees
- moved R1 152.4 mm to (91.0, 168.0), turned to 180 degrees
- moved R13 151.7 mm to (114.0, 187.0), turned to 180 degrees
- moved SW1 148.6 mm to (80.0, 168.0)
- moved R8 143.9 mm to (86.0, 182.0)
- moved J3 142.6 mm to (55.0, 89.0)
- moved J2 142.4 mm to (55.0, 74.0)
- moved D4 138.8 mm to (144.0, 179.0)
- moved D5 132.9 mm to (144.0, 184.0)
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Other:
- board outline added: 173 x 78 mm

Commit message: ready to route
Parts:
- added REF3: MountingHole_3mm_Pad_Via, Mounting_Holes:MountingHole_3mm_Pad_Via, F.Cu at (137.0, 58.0)
- added REF4: MountingHole_3mm_Pad_Via, Mounting_Holes:MountingHole_3mm_Pad_Via, F.Cu at (137.0, 126.0)
- moved R18 113.4 mm to (110.0, 71.0)
- moved U2 108.2 mm to (76.0, 64.0)
- moved D2 107.7 mm to (120.0, 64.0)
- moved R14 107.7 mm to (120.0, 69.0), turned to 180 degrees
- moved R6 107.6 mm to (91.0, 96.0), turned to 90 degrees
- moved R5 106.7 mm to (86.0, 96.0), turned to 90 degrees
- moved R4 106.2 mm to (81.0, 96.0), turned to 90 degrees
- moved R3 106.1 mm to (76.0, 96.0), turned to 90 degrees
- moved R19 104.0 mm to (110.0, 87.0)
- moved R15 104.0 mm to (120.0, 78.0), turned to 180 degrees
- moved TP1 102.6 mm to (65.0, 56.0)
- moved R10 102.1 mm to (110.0, 61.0), turned to 0 degrees
- moved R2 101.1 mm to (83.0, 83.0)
- moved Q1 98.7 mm to (110.0, 66.0)
- moved R11 95.1 mm to (110.0, 76.0), turned to 0 degrees
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- renumbered REF** to REF1, REF** to REF2
Routing:
- added copper zone on F.Cu, net +3V3
- added copper zone on F.Cu, net /5V
- added copper zone on F.Cu, net GND
Other:
- board size 173 x 78 mm -> 95 x 78 mm
- net class Default: clearance 0.2 -> 0.3; trace_width 0.25 -> 0.35; via_dia 0.6 -> 0.7; via_drill 0.4 -> 0.5
- rule trace_clearance: 0.2 -> 0.3

Commit message: small fix
Parts:
- moved R2 6.00 mm to (77.0, 83.0)
Changed lines of the file:
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@@
     (links 83)
     (no_connects 81)
-    (area 46.949999 52.949999 142.050001 131.050001)
+    (area 41.2 52.925 147.800001 131.175)
     (thickness 1.6)
     (drawings 4)
@@
     (pad_to_mask_clearance 0)
     (aux_axis_origin 0 0)
-    (visible_elements FFFFF77F)
+    (visible_elements FFFFFF7F)
     (pcbplotparams
       (layerselection 0x00030_80000001)
@@
   )
   (module Resistors_SMD:R_0805_HandSoldering (layer F.Cu)
-    (at 83 83)
+    (at 77 83)
     (descr "Resistor SMD 0805, hand soldering")
     (tags "resistor 0805")

Commit message: routed
Parts:
- moved J6 51.8 mm to (75.0, 65.0), turned to 90 degrees
- moved R15 21.5 mm to (101.0, 88.0)
- moved J1 20.0 mm to (120.5, 92.0)
- moved C1 20.0 mm to (112.2, 92.0)
- moved C2 20.0 mm to (112.2, 69.0)
- moved C3 20.0 mm to (112.2, 74.8)
- moved REF3 20.0 mm to (117.0, 58.0)
- moved REF4 20.0 mm to (117.0, 126.0)
- moved U1 20.0 mm to (112.2, 82.0)
- moved R14 19.0 mm to (101.0, 68.0)
- moved R16 19.0 mm to (101.0, 106.0)
- moved D2 19.0 mm to (101.0, 64.0)
- moved D3 19.0 mm to (101.0, 83.0)
- moved D4 19.0 mm to (101.0, 102.0)
- moved D5 19.0 mm to (101.0, 121.0)
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Connections:
- C1 pad 2: GND -> GNDD
- C2 pad 1: +3V3 -> VCC
- C2 pad 2: GND -> GNDD
- C3 pad 1: +3V3 -> VCC
- C3 pad 2: GND -> GNDD
- J1 pad 5: GND -> GNDD
- U1 pad 1: GND -> GNDD
- U1 pad 2: +3V3 -> VCC
Routing:
- net +3V3: track 0.00 -> 317.1 mm
- net /FLASH: track 0.00 -> 182.4 mm
- net /LED4_CTL: track 0.00 -> 152.9 mm
- net GND: track 0.00 -> 145.6 mm, vias 0 -> 2
- net /RESET: track 0.00 -> 131.5 mm
- net /BTN4: track 0.00 -> 123.9 mm
- net /XLED1: track 0.00 -> 115.7 mm
- net /BTN3: track 0.00 -> 88.1 mm
- net /XLED2: track 0.00 -> 66.3 mm
- net /LED1_CTL: track 0.00 -> 57.5 mm
- net /BTN1: track 0.00 -> 47.9 mm
- net /LED3_CTL: track 0.00 -> 43.3 mm
- net /XLED4: track 0.00 -> 40.3 mm
- net /XLED3: track 0.00 -> 39.6 mm
- net /BTN2: track 0.00 -> 26.0 mm
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Other:
- board size 95 x 78 mm -> 75 x 78 mm

Commit message: fixing PCB
Connections:
- C1 pad 2: GNDD -> GND
- C2 pad 1: VCC -> +3V3
- C2 pad 2: GNDD -> GND
- C3 pad 1: VCC -> +3V3
- C3 pad 2: GNDD -> GND
- J1 pad 5: GNDD -> GND
- U1 pad 1: GNDD -> GND
- U1 pad 2: VCC -> +3V3
Routing:
- net GND: track 145.6 -> 179.1 mm, vias 2 -> 4
- net +3V3: track 317.1 -> 342.5 mm, vias 0 -> 2
- net /5V: track 0.00 -> 11.6 mm
- net /PC_RX: track 17.5 -> 28.1 mm
- net /PC_TX: track 20.9 -> 28.1 mm
- net /BTN1: track 47.9 -> 49.5 mm
- added copper zone on F.Cu, net (none)
