File: hard/proj/controller.kicad_pcb (KiCad board)
At the start: 2 copper layers, 75 x 78 mm, 48 parts, among them J1 microUSB, J2 EXT1, J3 EXT2, J4 EXT3, J5 EXT4, J6 UART, Q1 BC848B, Q2 BC848B, Q3 BC848B, Q4 BC848B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

Commit message: PCB graphics
Parts:
- added G***: LOGO, Project-Lib:krol, F.Cu at (114.0, 112.5)
- added REF***: KiCad-Logo2_6mm_SilkScreen, Project-Lib:KiCad-Logo2_6mm_Copper, F.Cu at (80.5, 57.0)
- added REF***: OSHW-Logo_7.5x8mm_Copper, Symbols:OSHW-Logo_7.5x8mm_Copper, F.Cu at (69.0, 57.5)
- added VIA1: Measurement_Point_Round-SMD-Pad_Small, Wire_Pads:SolderWirePad_single_0-8mmDrill, F.Cu at (91.3, 72.3)
- added VIA2: Measurement_Point_Round-SMD-Pad_Small, Wire_Pads:SolderWirePad_single_0-8mmDrill, F.Cu at (81.0, 101.0)
- added VIA3: Measurement_Point_Round-SMD-Pad_Small, Wire_Pads:SolderWirePad_single_0-8mmDrill, F.Cu at (81.0, 113.5)
- added VIA5: Measurement_Point_Round-SMD-Pad_Small, Wire_Pads:SolderWirePad_single_0-8mmDrill, F.Cu at (102.9, 77.5)
- added VIA6: Measurement_Point_Round-SMD-Pad_Small, Wire_Pads:SolderWirePad_single_0-8mmDrill, F.Cu at (110.0, 72.2)
- added VIA7: Measurement_Point_Round-SMD-Pad_Small, Wire_Pads:SolderWirePad_single_0-8mmDrill, F.Cu at (115.2, 77.5)
- moved R3 3.00 mm to (75.0, 97.0)
- moved R4 3.00 mm to (72.0, 97.0)
Routing:
- net /BTN1: track 49.5 -> 41.4 mm
- net /RESET: track 131.5 -> 133.9 mm
- net GND: track 179.1 -> 178.1 mm
Other:
- net class Default: via_dia 0.7 -> 1.5; via_drill 0.5 -> 1
- board text added: "1"
- board text added: "2"
- board text added: "3"
- board text added: "4"
- board text added: "FLASH"
- board text added: "GND"
- board text added: "GitHub.com/ Himura2la/ AniQuiz"
- board text added: "RST"
- board text added: "TX"
- board text added: "tulafest.ru"

Commit message: fix DRC
Parts:
- removed VIA2: Measurement_Point_Round-SMD-Pad_Small, Wire_Pads:SolderWirePad_single_0-8mmDrill
Connections:
- VIA1 pad 1: (no net) -> GND
- VIA3 pad 1: (no net) -> GND
- VIA5 pad 1: (no net) -> +3V3
Routing:
- net GND: track 178.1 -> 214.4 mm, vias 4 -> 3
- net Net-(J1-Pad6): track 0.00 -> 12.3 mm
- net /5V: track 11.6 -> 17.5 mm
Changed lines of the file:
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@@
 (kicad_pcb (version 4) (host pcbnew 4.0.7)
   (general
-    (links 85)
-    (no_connects 8)
+    (links 88)
+    (no_connects 1)
     (area 46.949999 52.949999 122.050001 131.050001)
     (thickness 1.6)
     (drawings 18)
-    (tracks 1018)
+    (tracks 1033)
     (zones 0)
-    (modules 57)
+    (modules 56)
     (nets 37)
   )
@@
     (last_trace_width 0.35)
     (trace_clearance 0.3)
-    (zone_clearance 0.5)
+    (zone_clearance 0.508)
     (zone_45_only yes)
     (trace_min 0.2)
@@
       (effects (font (size 1 1) (thickness 0.15)))
     )
-    (pad 1 thru_hole circle (at 0 0) (size 1.99898 1.99898) (drill 0.8001) (layers *.Cu *.Mask))
+    (pad 1 thru_hole circle (at 0 0) (size 1.99898 1.99898) (drill 0.8001) (layers *.Cu *.Mask)
+      (net 3 +3V3))
   )
   (module Wire_Pads:SolderWirePad_single_0-8mmDrill (layer F.Cu)
@@
       (effects (font (size 1 1) (thickness 0.15)))
     )
-    (pad 1 thru_hole circle (at 0 0) (size 1.99898 1.99898) (drill 0.8001) (layers *.Cu *.Mask))
-  )
-  (module Wire_Pads:SolderWirePad_single_0-8mmDrill (layer F.Cu)
-    (at 81 101)
-    (fp_text reference VIA2 (at 0 -2.54) (layer F.SilkS) hide
-      (effects (font (size 1 1) (thickness 0.15)))
-    )
-    (fp_text value Measurement_Point_Round-SMD-Pad_Small (at 0 2.54) (layer F.Fab)
-      (effects (font (size 1 1) (thickness 0.15)))
-    )
-    (pad 1 thru_hole circle (at 0 0) (size 1.99898 1.99898) (drill 0.8001) (layers *.Cu *.Mask))
+    (pad 1 thru_hole circle (at 0 0) (size 1.99898 1.99898) (drill 0.8001) (layers *.Cu *.Mask)
+      (net 2 GND))
   )
   (module Wire_Pads:SolderWirePad_single_0-8mmDrill (layer F.Cu)
@@
       (effects (font (size 1 1) (thickness 0.15)))
     )
-    (pad 1 thru_hole circle (at 0 0) (size 1.99898 1.99898) (drill 0.8001) (layers *.Cu *.Mask))
+    (pad 1 thru_hole circle (at 0 0) (size 1.99898 1.99898) (drill 0.8001) (layers *.Cu *.Mask)
+      (net 2 GND))
   )
   (module Project-Lib:KiCad-Logo2_6mm_Copper (layer F.Cu)
@@
   (gr_line (start 47 131) (end 122 131) (angle 90) (layer Edge.Cuts) (width 0.1))
   (gr_line (start 47 131) (end 47 53) (angle 90) (layer Edge.Cuts) (width 0.1))
+  (segment (start 117.89 93.3) (end 112.95 93.3) (width 0.35) (layer F.Cu) (net 1))
+  (segment (start 112.95 93.3) (end 112.25 94) (width 0.35) (layer F.Cu) (net 1))
   (segment (start 109.1 84.3) (end 109.1 91.85) (width 0.35) (layer F.Cu) (net 1))
   (segment (start 111.25 94) (end 112.25 94) (width 0.35) (layer F.Cu) (net 1))
   (segment (start 109.1 91.85) (end 111.25 94) (width 0.35) (layer F.Cu) (net 1))
+  (segment (start 117.89 90.7) (end 112.95 90.7) (width 0.35) (layer F.Cu) (net 2))
+  (segment (start 112.95 90.7) (end 112.25 90) (width 0.35) (layer F.Cu) (net 2))
+  (segment (start 81 113.5) (end 81 103.6) (width 0.35) (layer B.Cu) (net 2))
+  (segment (start 90 73.6) (end 91.3 72.3) (width 0.35) (layer B.Cu) (net 2))
+  (segment (start 90 94.6) (end 90 73.6) (width 0.35) (layer B.Cu) (net 2))
+  (segment (start 81 103.6) (end 90 94.6) (width 0.35) (layer B.Cu) (net 2))
   (segment (start 81 98.35) (end 78 98.35) (width 0.35) (layer F.Cu) (net 2))
   (segment (start 78 98.35) (end 75 98.35) (width 0.35) (layer F.Cu) (net 2))
   (segment (start 75 98.35) (end 72 98.35) (width 0.35) (layer F.Cu) (net 2))
-  (segment (start 81 98.35) (end 81 101) (width 0.35) (layer F.Cu) (net 2))
   (via (at 110 72.25) (size 0.7) (drill 0.5) (layers F.Cu B.Cu) (net 2))
   (segment (start 91.1239 72.25) (end 91.25 72.25) (width 0.35) (layer F.Cu) (net 2))
@@
   (segment (start 68.41 113.41) (end 68.41 110) (width 0.35) (layer F.Cu) (net 2))
   (segment (start 68.5 113.5) (end 68.41 113.41) (width 0.35) (layer F.Cu) (net 2))
-  (segment (start 81 113.5) (end 68.5 113.5) (width 0.35) (layer F.Cu) (net 2))
+  (segment (start 81 113.5) (end 79 113.5) (width 0.35) (layer F.Cu) (net 2))
+  (segment (start 79 113.5) (end 68.5 113.5) (width 0.35) (layer F.Cu) (net 2))
   (via (at 81 113.5) (size 0.7) (drill 0.5) (layers F.Cu B.Cu) (net 2))
-  (segment (start 81 101) (end 81 113.5) (width 0.35) (layer B.Cu) (net 2))
-  (via (at 81 101) (size 0.7) (drill 0.5) (layers F.Cu B.Cu) (net 2))
   (segment (start 91.1724 97.1936) (end 90.9061 97.1936) (width 0.35) (layer F.Cu) (net 2))
   (segment (start 91.6411 96.7249) (end 91.1724 97.1936) (width 0.35) (layer F.Cu) (net 2))
@@
   (segment (start 101.775 116.475) (end 101.775 116.65) (width 0.35) (layer F.Cu) (net 9))
   (segment (start 102.35 116) (end 101.775 116.475) (width 0.35) (layer F.Cu) (net 9))
+  (segment (start 120.55 91.16) (end 120.55 92.84) (width 0.35) (layer F.Cu) (net 10) (status C00000))
+  (segment (start 118.25 89.0375) (end 120.4975 89.0375) (width 0.35) (layer F.Cu) (net 10))
+  (segment (start 120.4975 89.0375) (end 120.55 89.09) (width 0.35) (layer F.Cu) (net 10))
+  (segment (start 120.55 89.09) (end 120.55 92.84) (width 0.35) (layer F.Cu) (net 10))
+  (segment (start 120.55 92.84) (end 120.55 94.91) (width 0.35) (layer F.Cu) (net 10))
+  (segment (start 120.55 94.91) (end 120.4975 94.9625) (width 0.35) (layer F.Cu) (net 10))
+  (segment (start 120.4975 94.9625) (end 118.25 94.9625) (width 0.35) (layer F.Cu) (net 10))
+  (segment (start 120.4975 89.0375) (end 120.55 89.09) (width 0.35) (layer F.Cu) (net 10))
+  (segment (start 120.55 94.91) (end 120.4975 94.9625) (width 0.35) (layer F.Cu) (net 10))
   (segment (start 54.4253 74) (end 55 74) (width 0.35) (layer F.Cu) (net 11))
   (segment (start 54.4253 84.8774) (end 54.4253 74) (width 0.35) (layer F.Cu) (net 11))
@@
   )
   (zone (net 0) (net_name "") (layer F.Cu) (hatch edge 0.508)
-    (connect_pads (clearance 0.508))
-    (min_thickness 0.254)
-    (keepout (tracks allowed) (vias allowed) (copperpour not_allowed))
-    (fill (arc_segments 16) (thermal_gap 0.508) (thermal_bridge_width 0.508))
-    (polygon
-      (pts
-        (xy 117.8 71.1) (xy 115.8 73.1) (xy 115.8 75.7) (xy 116.9 77) (xy 116.9 84.5)
-        (xy 113.5 84.5) (xy 113.5 88.5) (xy 116.5 88.5) (xy 116.5 87.25) (xy 122.5 87.25)
-        (xy 122.5 97) (xy 122 97) (xy 122 123) (xy 105 123) (xy 105 120)
-        (xy 107 118) (xy 107 114) (xy 106 113) (xy 106 96.25) (xy 111.5 96.25)
-        (xy 107.5 92.25) (xy 107.5 77) (xy 108.75 75.75) (xy 108.7 73.3) (xy 106.8 71.4)
-        (xy 106.7 67.2) (xy 117.8 67.2)
-      )
-    )
-  )
-  (zone (net 0) (net_name "") (layer F.Cu) (hatch edge 0.508)
     (connect_pads no (clearance 0.5))
     (min_thickness 1.4)
@@
     (polygon
       (pts
-        (xy 122 131) (xy 47 131) (xy 47 53) (xy 122 53)
+        (xy 122 131) (xy 47 131) (xy 47 53) (xy 122 53) (xy 122 66.4)
+        (xy 122 87.2) (xy 117 87.2) (xy 117 76.4) (xy 115.8 75.2) (xy 115.8 73.6)
+        (xy 118.2 71.2) (xy 118.2 66.4) (xy 106.4 66.4) (xy 106.4 71.4) (xy 108.4 73.4)
+        (xy 108.4 75.6) (xy 107 77) (xy 107 122.6) (xy 122 122.6)
       )
     )
@@
     (connect_pads (clearance 0.508))
     (min_thickness 0.254)
-    (keepout (tracks not_allowed) (vias not_allowed) (copperpour not_allowed))
+    (keepout (tracks allowed) (vias allowed) (copperpour not_allowed))
     (fill (arc_segments 16) (thermal_gap 0.508) (thermal_bridge_width 0.508))
     (polygon
