File: hard/proj/controller.kicad_pcb (KiCad board)
At the start: 2 copper layers, 44 parts, among them J1 microUSB, J2 EXT1, J3 EXT2, J4 EXT3, J5 EXT4, J6 UART, Q1 BC848B, Q2 BC848B, Q3 BC848B, Q4 BC848B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

Commit message: layouted
Parts:
- added M1: MountingHole_3mm_Pad_Via, MountingHole:MountingHole_3mm_Pad_Via, F.Cu at (36.0, 92.5)
- added M2: MountingHole_3mm, MountingHole:MountingHole_3mm, F.Cu at (63.0, 92.5)
- added M3: MountingHole_3mm_Pad_Via, MountingHole:MountingHole_3mm_Pad_Via, F.Cu at (63.0, 154.5)
- added M4: MountingHole_3mm_Pad_Via, MountingHole:MountingHole_3mm_Pad_Via, F.Cu at (36.0, 154.5)
- moved R18 150.4 mm to (34.4, 98.2), turned to 180 degrees
- moved R19 140.3 mm to (34.2, 111.8), turned to 180 degrees
- moved R20 138.7 mm to (38.5, 128.0)
- moved R13 134.4 mm to (50.0, 148.8), turned to 180 degrees
- moved R5 134.2 mm to (38.5, 135.2)
- moved R21 128.6 mm to (38.5, 141.5)
- moved R10 128.4 mm to (50.0, 130.5), turned to 180 degrees
- moved Q2 125.9 mm to (54.5, 137.5)
- moved Q3 125.7 mm to (54.5, 143.5)
- moved R2 125.7 mm to (45.2, 105.0)
- moved TP1 125.2 mm to (42.2, 103.2)
- moved R3 121.1 mm to (38.5, 108.2)
- moved R8 119.7 mm to (53.5, 120.1), turned to 180 degrees
- moved R12 118.7 mm to (50.0, 142.5), turned to 180 degrees
- moved D2 117.8 mm to (59.0, 133.0), turned to 180 degrees
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Connections:
- J1 pad 6: Net-(J1-Pad6) -> (no net)
Other:
- board outline added: 35 x 70 mm
- board text added: "1"
- board text added: "2"
- board text added: "3"
- board text added: "4"
- board text added: "FLASH"
- board text added: "G"
- board text added: "R"
- board text added: "RESET"
- board text added: "T"

Commit message: routing
Parts:
- TP1: moved to B.Cu
- moved J6 68.4 mm to (40.9, 90.3), turned to 270 degrees
- moved R18 7.48 mm to (41.8, 97.1), turned to 90 degrees
- moved TP1 6.71 mm to (41.8, 96.5)
- moved R3 4.97 mm to (42.7, 110.9), turned to 90 degrees
- moved R20 2.40 mm to (40.9, 128.0)
- moved C1 1.65 mm to (58.8, 126.0)
- moved R7 1.61 mm to (58.8, 121.0)
- moved R19 1.29 mm to (35.3, 111.0), turned to 90 degrees
- moved D1 0.60 mm to (56.4, 120.1), turned to 0 degrees
- moved R8 0.30 mm to (53.2, 120.1)
- moved R9 0.23 mm to (49.8, 120.1)
Routing:
- net +3V3: track 0.00 -> 149.6 mm, vias 0 -> 1
- net GND: track 0.00 -> 144.2 mm
- net /FLASH: track 0.00 -> 85.2 mm, vias 0 -> 1
- net /LED2_PWR: track 0.00 -> 84.5 mm, vias 0 -> 2
- net /LED1_PWR: track 0.00 -> 53.9 mm, vias 0 -> 2
- net /LED4_CTL: track 0.00 -> 48.2 mm, vias 0 -> 1
- net /LED3_CTL: track 0.00 -> 46.1 mm, vias 0 -> 1
- net /LED1_CTL: track 0.00 -> 45.5 mm, vias 0 -> 1
- net /LED2_CTL: track 0.00 -> 44.1 mm, vias 0 -> 1
- net /BTN4: track 0.00 -> 41.1 mm
- net /RESET: track 0.00 -> 38.5 mm, vias 0 -> 1
- net /BTN3: track 0.00 -> 29.2 mm
- net /PC_TX: track 0.00 -> 28.3 mm
- net /PC_RX: track 0.00 -> 25.7 mm
- net /LED3_PWR: track 0.00 -> 25.3 mm
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Other:
- net class Default: clearance 0.2 -> 0.3; trace_width 0.25 -> 0.4; via_dia 0.8 -> 1; via_drill 0.4 -> 0.8
- net class Power added: clearance 0.3, trace_width 0.6, via_dia 1, via_drill 0.8
- net class Signal added: clearance 0.3, trace_width 0.3, via_dia 1, via_drill 0.8
- rule trace_clearance: 0.2 -> 0.3
- rule trace_min: 0.2 -> 0.3
- rule via_min_drill: 0.3 -> 0.8
- rule via_min_size: 0.4 -> 0.8
- board text added: "3.3V"

Commit message: routed
Parts:
- moved R17 5.03 mm to (57.5, 153.8)
Routing:
- net GND: track 144.2 -> 215.9 mm, vias 0 -> 1
- net +3V3: track 149.6 -> 217.7 mm, vias 1 -> 2
- net /LED4_PWR: track 23.0 -> 36.3 mm
- net /LED1_CTL: track 45.5 -> 43.4 mm
- net Net-(D5-Pad1): track 1.91 -> 3.01 mm
- net /PC_RX: track 25.7 -> 26.7 mm
- net /LED3_CTL: track 46.1 -> 45.1 mm
- net /LED3_PWR: track 25.3 -> 26.3 mm
- net /FLASH: track 85.2 -> 84.4 mm
- net /LED4_CTL: track 48.2 -> 47.4 mm
Other:
- board text added: "RST"
- board text removed: "RESET"

Commit message: zones+symbols
Parts:
- added REF**: KiCad-Logo_6mm_SilkScreen, Project-Lib:KiCad-Logo_3mm_Copper, B.Cu at (56.0, 110.8)
Routing:
- net GND: track 215.9 -> 215.4 mm
- added copper zone on B.Cu, net +3V3
- added copper zone on B.Cu, net GND
- added copper zone on F.Cu, net GND
Other:
- board text added: "github.com/ Himura2la/AniQuiz"
- board text added: "tulafest.ru"

Commit message: errors (((
Parts:
- moved TP1 2.90 mm to (39.0, 95.8)
Routing:
- net /ADC: track 12.9 -> 16.0 mm
- net /FLASH: track 84.4 -> 85.6 mm
- net GND: track 215.4 -> 215.9 mm
Changed lines of the file:
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@@
     (thickness 1.6)
     (drawings 20)
-    (tracks 360)
+    (tracks 362)
     (zones 0)
     (modules 49)
@@
     (0 F.Cu signal)
     (31 B.Cu signal)
-    (32 B.Adhes user)
-    (33 F.Adhes user)
-    (34 B.Paste user)
+    (32 B.Adhes user hide)
+    (33 F.Adhes user hide)
+    (34 B.Paste user hide)
     (35 F.Paste user hide)
     (36 B.SilkS user hide)
-    (37 F.SilkS user)
+    (37 F.SilkS user hide)
     (38 B.Mask user hide)
     (39 F.Mask user hide)
@@
     (46 B.CrtYd user hide)
     (47 F.CrtYd user hide)
-    (48 B.Fab user hide)
-    (49 F.Fab user hide)
+    (48 B.Fab user)
+    (49 F.Fab user)
   )
   (setup
@@
       (drillshape 1)
       (scaleselection 1)
-      (outputdirectory ""))
+      (outputdirectory C:/Users/glago/Desktop/))
   )
   (net 0 "")
@@
   )
   (module TestPoint:TestPoint_Pad_D1.5mm (layer B.Cu)
-    (at 41.8 96.5)
+    (at 39 95.75)
     (descr "SMD pad as test Point, diameter 1.5mm")
     (tags "test point SMD pad")
@@
   )
   (gr_text "github.com/\nHimura2la/AniQuiz" (at 49 156.25) (layer F.Cu)
-    (effects (font (size 1 1) (thickness 0.25)))
+    (effects (font (size 1 1.3) (thickness 0.25)))
   )
   (gr_text 3.3V (at 38.5 102) (layer F.Cu)
@@
   (segment (start 64.9 138.69) (end 64.9 140.1) (width 1) (layer F.Cu) (net 1))
   (segment (start 60.6 118.4) (end 60.6 122.1) (width 0.7) (layer F.Cu) (net 1))
-  (segment (start 64 117) (end 62 117) (width 0.7) (layer F.Cu) (net 1))
+  (segment (start 64 117) (end 62 117) (width 1.5) (layer F.Cu) (net 1))
   (segment (start 62 117) (end 60.6 118.4) (width 0.7) (layer F.Cu) (net 1))
   (segment (start 48.52 95.927122) (end 48.52 91.502081) (width 0.4) (layer B.Cu) (net 1))
@@
   (segment (start 61.2 103.4) (end 55.992878 103.4) (width 0.4) (layer B.Cu) (net 1))
   (segment (start 62.8 101.8) (end 61.2 103.4) (width 0.4) (layer B.Cu) (net 1))
-  (segment (start 65.2 117) (end 65.2 118) (width 0.8) (layer B.Cu) (net 1))
-  (segment (start 65.2 118) (end 65.2 119) (width 0.8) (layer B.Cu) (net 1))
-  (segment (start 65.2 119) (end 66 119.8) (width 0.8) (layer B.Cu) (net 1))
-  (segment (start 66 141) (end 65.8 141) (width 0.3) (layer B.Cu) (net 1))
-  (segment (start 66.2 119.8) (end 66.2 140.8) (width 0.3) (layer B.Cu) (net 1))
-  (segment (start 66.2 140.8) (end 66 141) (width 0.3) (layer B.Cu) (net 1))
+  (segment (start 66.2 119.2) (end 64 117) (width 0.3) (layer B.Cu) (net 1))
+  (segment (start 66.2 140.8) (end 66.2 119.2) (width 0.3) (layer B.Cu) (net 1))
+  (segment (start 65.8 141) (end 66 141) (width 0.3) (layer B.Cu) (net 1))
+  (segment (start 66 141) (end 66.2 140.8) (width 0.3) (layer B.Cu) (net 1))
   (segment (start 50.85 127.3) (end 49.35 127.3) (width 0.6) (layer F.Cu) (net 2))
   (segment (start 52.35 128.8) (end 50.85 127.3) (width 0.6) (layer F.Cu) (net 2))
@@
   (segment (start 55.52 120.1) (end 54.1675 120.1) (width 1) (layer F.Cu) (net 4))
   (segment (start 57.28 120.1) (end 58.7325 120.1) (width 1) (layer F.Cu) (net 5))
-  (segment (start 58.8 116.2) (end 64 111) (width 0.9) (layer F.Cu) (net 5))
-  (segment (start 58.8 120.0325) (end 58.8 116.2) (width 0.9) (layer F.Cu) (net 5))
   (via (at 65.4 149.3) (size 2) (drill 0.8) (layers F.Cu B.Cu) (net 5))
   (segment (start 65.4 149.3) (end 63.61 149.3) (width 1.5) (layer F.Cu) (net 5))
@@
   (segment (start 60.6 114.4) (end 60.6 119.1) (width 0.3) (layer B.Cu) (net 5))
   (segment (start 54.3 142.2) (end 50.5 142.2) (width 0.3) (layer B.Cu) (net 5))
+  (segment (start 61.95 111) (end 64 111) (width 1.5) (layer F.Cu) (net 5))
+  (segment (start 58.8 120.0325) (end 58.8 114.15) (width 0.9) (layer F.Cu) (net 5))
+  (segment (start 58.8 114.15) (end 61.95 111) (width 0.9) (layer F.Cu) (net 5))
   (segment (start 59.88 130.95625) (end 59.88 132.86875) (width 0.8) (layer F.Cu) (net 6))
   (segment (start 59.88 137) (end 59.88 138.9125) (width 0.8) (layer F.Cu) (net 7))
@@
   (segment (start 64 115) (end 62.6 116.4) (width 0.3) (layer B.Cu) (net 42))
   (segment (start 51.599999 147.900001) (end 51.599999 149.750019) (width 0.3) (layer B.Cu) (net 42))
-  (segment (start 41.8 99.5) (end 41.8 97.1) (width 0.8) (layer B.Cu) (net 43))
   (segment (start 50 105) (end 47.3 105) (width 0.8) (layer B.Cu) (net 43))
   (segment (start 47.3 105) (end 41.8 99.5) (width 0.8) (layer B.Cu) (net 43))
+  (segment (start 40.06066 95.75) (end 39 95.75) (width 0.8) (layer B.Cu) (net 43))
+  (segment (start 40.110002 95.75) (end 40.06066 95.75) (width 0.8) (layer B.Cu) (net 43))
+  (segment (start 41.8 97.439998) (end 40.110002 95.75) (width 0.8) (layer B.Cu) (net 43))
+  (segment (start 41.8 99.5) (end 41.8 97.439998) (width 0.8) (layer B.Cu) (net 43))
   (zone (net 0) (net_name "") (layers F&B.Cu) (hatch full 0.508)
     (connect_pads (clearance 0.508))
@@
     (polygon
       (pts
-        (xy 59.8 125.25) (xy 63.9 125.25) (xy 63.9 121.45) (xy 59.8 121.45)
+        (xy 56.9 126.5) (xy 63.9 126.45) (xy 63.9 120.1) (xy 56.9 120.15)
       )
     )
@@
       )
     )
+  )
+  (zone (net 0) (net_name "") (layer B.Cu) (hatch edge 0.508)
+    (connect_pads (clearance 0.5))
+    (min_thickness 0.254)
+    (keepout (tracks allowed) (vias allowed) (copperpour not_allowed))
+    (fill (arc_segments 16) (thermal_gap 0.508) (thermal_bridge_width 0.508))
+    (polygon
+      (pts
+        (xy 36 88.5) (xy 36 90.5) (xy 41.25 90.5) (xy 41.25 88.5)
+      )
+    )
+  )
+  (zone (net 0) (net_name "") (layer B.Cu) (hatch edge 0.508)
+    (connect_pads (clearance 0.5))
+    (min_thickness 0.254)
+    (keepout (tracks allowed) (vias allowed) (copperpour not_allowed))
+    (fill (arc_segments 16) (thermal_gap 0.508) (thermal_bridge_width 0.508))
+    (polygon
+      (pts
+        (xy 67 116) (xy 67 121) (xy 65 121) (xy 62 118) (xy 62 116)
+      )
+    )
+  )
+  (zone (net 0) (net_name "") (layer F.Cu) (hatch edge 0.508)
+    (connect_pads (clearance 0.5))
+    (min_thickness 0.254)
+    (keepout (tracks allowed) (vias allowed) (copperpour not_allowed))
+    (fill (arc_segments 16) (thermal_gap 0.508) (thermal_bridge_width 0.508))
+    (polygon
+      (pts
+        (xy 55.8 134.5) (xy 54 134.5) (xy 54 132) (xy 55.8 132)
+      )
+    )
+  )
+  (zone (net 0) (net_name "") (layer F.Cu) (hatch edge 0.508)
+    (connect_pads (clearance 0.5))
+    (min_thickness 0.254)
+    (keepout (tracks allowed) (vias allowed) (copperpour not_allowed))
+    (fill (arc_segments 16) (thermal_gap 0.508) (thermal_bridge_width 0.508))
+    (polygon
+      (pts
+        (xy 51.9 129.9) (xy 47.9 129.9) (xy 47.9 128) (xy 51.9 128)
+      )
+    )
+  )
+  (zone (net 0) (net_name "") (layer F.Cu) (hatch edge 0.508)
+    (connect_pads (clearance 0.5))
+    (min_thickness 0.254)
+    (keepout (tracks allowed) (vias allowed) (copperpour not_allowed))
+    (fill (arc_segments 16) (thermal_gap 0.508) (thermal_bridge_width 0.508))
+    (polygon
+      (pts
+        (xy 55.5 145.35) (xy 53.8 145.35) (xy 53.8 143.95) (xy 55.5 143.95)
+      )
+    )

Commit message: fixing errors
Parts:
- removed D1: STATUS, LED_SMD:LED_0805_2012Metric_Pad1.12x1.40mm_HandSolder
- R8, R9: value 180 -> 10k
- moved R7 6.85 mm to (52.0, 120.2), turned to 180 degrees
- moved R9 5.80 mm to (55.6, 120.2)
- moved R8 5.67 mm to (58.8, 121.0), turned to 90 degrees
Connections:
- net /PC_RX renamed /UART_TX
- net /PC_TX renamed /UART_RX
- R7 pad 1: /FLASH -> +3V3
- R7 pad 2: +3V3 -> /FLASH
- R8 pad 1: Net-(D1-Pad1) -> GND
- R8 pad 2: Net-(R8-Pad2) -> /LED4_CTL
- R9 pad 1: GND -> +3V3
- R9 pad 2: Net-(R8-Pad2) -> /LED3_CTL
Routing:
- net /LED3_CTL: track 45.1 -> 56.6 mm
- net /LED4_CTL: track 47.4 -> 55.8 mm
- net /FLASH: track 85.6 -> 89.2 mm
- net GND: track 215.9 -> 218.0 mm
- net +3V3: track 217.7 -> 215.8 mm
- net Net-(R8-Pad2): track 1.47 -> 0.00 mm
- net Net-(D1-Pad1): track 1.35 -> 0.00 mm

Commit message: fixing errors
Connections:
- R7 pad 2: /FLASH -> /LED3_CTL
- R9 pad 2: /LED3_CTL -> /GPIO2_HIGH
- SW2 pad 2: /FLASH -> /LED3_CTL
- U2 pad 11: /LED3_CTL -> /GPIO2_HIGH
- U2 pad 12: /FLASH -> /LED3_CTL
Routing:
- net /FLASH: track 89.2 -> 0.00 mm, vias 1 -> 0
- net /LED3_CTL: track 56.6 -> 91.1 mm, vias 1 -> 2
- net /GPIO2_HIGH: track 0.00 -> 11.7 mm
- net /XLED2: track 3.03 -> 2.23 mm
- net /LED1_CTL: track 43.4 -> 44.1 mm
- net /LED2_CTL: track 44.1 -> 44.7 mm
